File: kicad-fuse.kicad_pcb (KiCad board)
At the start: 2 copper layers, 22.4 x 9.4 mm, 3 parts, among them J1 Conn_01x02_Male

Commit message: Saved files in KiCad 7.
Other:
- board text added: "11-May-23"
- board text added: "Fuseholder v1.1d"
- board text removed: "1-Feb-23"
- board text removed: "Fuseholder v1.1b"
